Commit message: changed rotation

File: franka_description/robots/common/franka_suction.urdf.xacro (robot description, xacro)
@@ -3,5 +3,5 @@
 	name="schmalz_cobot_pump">
 	<xacro:property name="origin_xyz" value="0.0 0.0 0.0"/>
-	<xacro:property name="origin_rpy" value="0.0 0.0 0.0"/>
+	<xacro:property name="origin_rpy" value="3.1415 0.0 3.1415"/>
 	<xacro:macro name="franka_suction" params="path_prefix parent">
 		<joint name="vacuum_joint8" type="fixed">
@@ -13,15 +13,13 @@
 			<visual>
 				<geometry>
-					<mesh filename="package://${path_prefix}/robots/common/schmalz_cobot.stl"/>
+					<mesh filename="package://${path_prefix}/robots/common/schmalz_cobot.stl" scale="0.001 0.001 0.001"/>
 				</geometry>
 				<!-- might have to change this later if it looks weird in rviz-->
-				<origin xyz="${origin_xyz}" rpy="${origin_rpy}" />
 			</visual>
 			<collision>
 				<!-- if too slow change to cylinder -->
 				<geometry>
-					<mesh filename="package://${path_prefix}/robots/common/schmalz_cobot.stl"/>
+					<mesh filename="package://${path_prefix}/robots/common/schmalz_cobot.stl" scale="0.001 0.001 0.001"/>
                                 </geometry>
-				<origin xyz="${origin_xyz}" rpy="${origin_rpy}" />
 			</collision>
 			<inertial>
@@ -29,5 +27,4 @@
 				<mass value="0.775"/>
 				<inertia ixx="0.0016" ixy="0.0" ixz = "0.0" iyy="0.0016" iyz="0.0" izz="0.0009"/>
-				<origin xyz="${origin_xyz}" rpy="${origin_rpy}" />
 			</inertial>
 		</link>

Commit message: changed rotation

File: franka_description/robots/common/franka_suction.urdf.xacro (robot description, xacro)
@@ -3,5 +3,5 @@
 	name="schmalz_cobot_pump">
 	<xacro:property name="origin_xyz" value="0.0 0.0 0.0"/>
-	<xacro:property name="origin_rpy" value="0.0 0.0 0.0"/>
+	<xacro:property name="origin_rpy" value="3.1415 0.0 3.1415"/>
 	<xacro:macro name="franka_suction" params="path_prefix parent">
 		<joint name="vacuum_joint8" type="fixed">

Commit message: fixing rotation

File: franka_description/robots/common/franka_suction.urdf.xacro (robot description, xacro)
@@ -3,5 +3,5 @@
 	name="schmalz_cobot_pump">
 	<xacro:property name="origin_xyz" value="0.0 0.0 0.0"/>
-	<xacro:property name="origin_rpy" value="3.1415 0.0 3.1415"/>
+	<xacro:property name="origin_rpy" value="3.1415 0.0 3.25"/>
 	<xacro:macro name="franka_suction" params="path_prefix parent">
 		<joint name="vacuum_joint8" type="fixed">

Commit message: adding cylinders to base

File: franka_description/robots/common/franka_suction.urdf.xacro (robot description, xacro)
@@ -3,5 +3,5 @@
 	name="schmalz_cobot_pump">
 	<xacro:property name="origin_xyz" value="0.0 0.0 0.0"/>
-	<xacro:property name="origin_rpy" value="3.1415 0.0 3.25"/>
+	<xacro:property name="origin_rpy" value="3.1415 0.0 0.8"/>
 	<xacro:macro name="franka_suction" params="path_prefix parent">
 		<joint name="vacuum_joint8" type="fixed">
@@ -15,5 +15,4 @@
 					<mesh filename="package://${path_prefix}/robots/common/schmalz_cobot.stl" scale="0.001 0.001 0.001"/>
 				</geometry>
-				<!-- might have to change this later if it looks weird in rviz-->
 			</visual>
 			<collision>
@@ -29,4 +28,40 @@
 			</inertial>
 		</link>
+		<joint name="vacuum_joint9" type="fixed">
+			<parent link="vacuum"/>
+			<child link="cylinder1"/>
+			<origin xyz="${origin_xyz}" rpy="0.0 0.0 0.0" />
+		</joint>
+		<!-- wider cylinder at base of vacuum -->
+		<link name="cylinder1">
+			<visual>
+				<geometry>
+					<cylinder radius="0.025" length="0.0065"/>
+				</geometry>
+			</visual>
+			<collision>
+				<geometry>
+					<cylinder radius="0.025" length="0.0065"/>
+                                </geometry>
+			</collision>
+		</link>
+		<joint name="vacuum_joint10" type="fixed">
+                        <parent link="cylinder1"/>
+                        <child link="cylinder2"/>
+                        <origin xyz="${origin_xyz}" rpy="0.0 0.0 0.0" />
+                </joint>
+                <!-- thinner small cylinder at base of vacuum attached to the green gripper-->
+                <link name="cylinder2">
+                        <visual>
+                                <geometry>
+					<cylinder radius="0.005" length="0.0125"/>
+                                </geometry>
+                        </visual>
+                        <collision>
+                                <geometry>
+					<cylinder radius="0.005" length="0.0125"/>
+                                </geometry>
+                        </collision>
+                </link>
 	</xacro:macro>
 </robot>

Commit message: fixed cylinders and added reference point

File: franka_description/robots/common/franka_suction.urdf.xacro (robot description, xacro)
@@ -31,5 +31,5 @@
 			<parent link="vacuum"/>
 			<child link="cylinder1"/>
-			<origin xyz="${origin_xyz}" rpy="0.0 0.0 0.0" />
+			<origin xyz="0.0 0.0 -0.09" rpy="0.0 0.0 0.0" />
 		</joint>
 		<!-- wider cylinder at base of vacuum -->
@@ -49,5 +49,5 @@
                         <parent link="cylinder1"/>
                         <child link="cylinder2"/>
-                        <origin xyz="${origin_xyz}" rpy="0.0 0.0 0.0" />
+                        <origin xyz="0.0 0.0 -0.0065" rpy="0.0 0.0 0.0" />
                 </joint>
                 <!-- thinner small cylinder at base of vacuum attached to the green gripper-->
@@ -63,5 +63,13 @@
                                 </geometry>
                         </collision>
-                </link>
+		</link>
+		<joint name="vacuum_joint11" tpe="fixed">
+			<parent link="cylinder2"/>
+                        <child link="referencePoint"/>
+                        <origin xyz="0.0 0.0 -0.0125" rpy="0.0 0.0 0.0" />
+		</joint>
+		<!-- reference point at bottom of cylinder2 representing where the suction gripper is -->
+		<link name="referencePoint">
+		</link>
 	</xacro:macro>
 </robot>

Commit message: fixed cylinders and added reference point

File: franka_description/robots/common/franka_suction.urdf.xacro (robot description, xacro)
@@ -64,5 +64,5 @@
                         </collision>
 		</link>
-		<joint name="vacuum_joint11" tpe="fixed">
+		<joint name="vacuum_joint11" type="fixed">
 			<parent link="cylinder2"/>
                         <child link="referencePoint"/>
